File: ECU/EMControl.kicad_sch (KiCad schematic)
At the start: 5 parts, among them J1 Conn_01x20_Pin, J2 Conn_01x20_Pin, U8 NCP1117-3.3_SOT223

Commit message: VIO added
Connections:
- net VIO3: now reaches J2.5 (Pin_5)
- net VIO2: now reaches J2.6 (Pin_6)
- net VIO1: now reaches J2.7 (Pin_7)
- net VIO0: now reaches J2.8 (Pin_8)
Changed lines of the file:
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@@
+	(wire
+		(pts
+			(xy 153.67 35.56) (xy 189.23 35.56)
+		)
+		(stroke
+			(width 0)
+			(type default)
+		)
+	)
 	(wire
 		(pts
@@
 	(wire
 		(pts
+			(xy 153.67 38.1) (xy 189.23 38.1)
+		)
+		(stroke
+			(width 0)
+			(type default)
+		)
+	)
+	(wire
+		(pts
 			(xy 90.17 27.94) (xy 90.17 41.91)
 		)
@@
 	(wire
 		(pts
+			(xy 153.67 33.02) (xy 189.23 33.02)
+		)
+		(stroke
+			(width 0)
+			(type default)
+		)
+	)
+	(wire
+		(pts
 			(xy 153.67 71.12) (xy 153.67 143.51)
 		)
@@
 		(pts
 			(xy 156.21 148.59) (xy 156.21 68.58)
+		)
+		(stroke
+			(width 0)
+			(type default)
+		)
+	)
+	(wire
+		(pts
+			(xy 153.67 40.64) (xy 189.23 40.64)
 		)
 		(stroke
@@
 		)
 	)
+	(hierarchical_label "VIO1"
+		(shape input)
+		(at 189.23 38.1 0)
+		(effects
+			(font
+				(size 1.27 1.27)
+			)
+			(justify left)
+		)
+	)
 	(hierarchical_label "CIN9"
 		(shape input)
@@
 		)
 	)
+	(hierarchical_label "VIO0"
+		(shape input)
+		(at 189.23 40.64 0)
+		(effects
+			(font
+				(size 1.27 1.27)
+			)
+			(justify left)
+		)
+	)
+	(hierarchical_label "VIO2"
+		(shape input)
+		(at 189.23 35.56 0)
+		(effects
+			(font
+				(size 1.27 1.27)
+			)
+			(justify left)
+		)
+	)
 	(hierarchical_label "5V"
 		(shape input)
@@
 		)
 	)
+	(hierarchical_label "VIO3"
+		(shape input)
+		(at 189.23 33.02 0)
+		(effects
+			(font
+				(size 1.27 1.27)
+			)
+			(justify left)
+		)
+	)
